Commit message: fix(description): 统一 WL 驱动关节命名
原因：对齐 legged_control 控制器期望的 LF/LH/RF/RH + HAA/HFE/KFE 驱动关节命名，避免加载 HybridJointHandle 时找不到关节。

影响范围：仅修改 WL URDF 中 12 个 revolute 驱动关节的 name 属性，不调整 link、固定关节、足端、IMU、transmission 或 Gazebo 配置。

验证：使用 rg 确认 12 个 LF/LH/RF/RH 驱动关节名齐全，旧的 hip/thigh/calf_joint 驱动关节名已不存在。

File: legged_examples/legged_wl/legged_wl_description/urdf/wl.urdf (robot description, URDF)
Before this commit: robot a1_description, 23 links, 22 joints
Joints:
- removed joint FL_calf_joint
- removed joint FL_hip_joint
- removed joint FL_thigh_joint
- removed joint FR_calf_joint
- removed joint FR_hip_joint
- removed joint FR_thigh_joint
- removed joint RL_calf_joint
- removed joint RL_hip_joint
- removed joint RL_thigh_joint
- removed joint RR_calf_joint
- removed joint RR_hip_joint
- removed joint RR_thigh_joint
- added joint LF_HAA: type revolute, parent trunk, child FL_hip, origin xyz=0.1995 0.05001 0 rpy=0 0 0, axis 1 0 0, limit lower=-0.94 upper=0.94 effort=18 velocity=40
- added joint LF_HFE: type revolute, parent FL_hip, child FL_thigh, origin xyz=0 0.08505 0 rpy=0 0 0, axis 0 1 0, limit lower=-0.409203673 upper=3.550796326 effort=18 velocity=40
- added joint LF_KFE: type revolute, parent FL_thigh, child FL_calf, origin xyz=0 -0.0001 -0.2 rpy=0 0 0, axis 0 1 0, limit lower=-2.6 upper=-0.885 effort=50 velocity=26.6
- added joint LH_HAA: type revolute, parent trunk, child RL_hip, origin xyz=-0.1995 0.04999 0 rpy=0 0 0, axis 1 0 0, limit lower=-0.94 upper=0.94 effort=18 velocity=40
- added joint LH_HFE: type revolute, parent RL_hip, child RL_thigh, origin xyz=0 0.08985 0 rpy=0 0 0, axis 0 1 0, limit lower=-0.409203673 upper=3.550796326 effort=18 velocity=40
- added joint LH_KFE: type revolute, parent RL_thigh, child RL_calf, origin xyz=0 0.0001 -0.2 rpy=0 0 0, axis 0 1 0, limit lower=-2.6 upper=-0.885 effort=50 velocity=26.6
- added joint RF_HAA: type revolute, parent trunk, child FR_hip, origin xyz=0.1995 -0.05001 0 rpy=0 0 0, axis 1 0 0, limit lower=-0.94 upper=0.94 effort=18 velocity=40
- added joint RF_HFE: type revolute, parent FR_hip, child FR_thigh, origin xyz=0 -0.08505 0 rpy=0 0 0, axis 0 1 0, limit lower=-0.409203673 upper=3.550796326 effort=18 velocity=40
- added joint RF_KFE: type revolute, parent FR_thigh, child FR_calf, origin xyz=0 -0.0001 -0.2 rpy=0 0 0, axis 0 1 0, limit lower=-2.6 upper=-0.885 effort=50 velocity=26.6
- added joint RH_HAA: type revolute, parent trunk, child RR_hip, origin xyz=-0.1995 -0.05001 0 rpy=0 0 0, axis 1 0 0, limit lower=-0.94 upper=0.94 effort=18 velocity=40
- added joint RH_HFE: type revolute, parent RR_hip, child RR_thigh, origin xyz=0 -0.08985 0 rpy=0 0 0, axis 0 1 0, limit lower=-0.409203673 upper=3.550796326 effort=18 velocity=40
- added joint RH_KFE: type revolute, parent RR_thigh, child RR_calf, origin xyz=0 -0.0001 -0.2 rpy=0 0 0, axis 0 1 0, limit lower=-2.6 upper=-0.885 effort=50 velocity=26.6

Commit message: fix(description): 统一 WL 足端命名
原因：对齐 legged_control 常用的 LF/LH/RF/RH_FOOT 足端 contact frame 命名，为后续 OCS2 contactNames3DoF 和 Gazebo contact 配置适配做准备。

影响范围：仅修改 WL URDF 中 4 个足端 link、child link 引用和对应 foot fixed joint 名称，不调整小腿 link、几何、惯量、contact 配置或控制参数。

验证：使用 rg 确认 LF/LH/RF/RH_FOOT 均存在，旧的 FL/FR/RL/RR_foot 名称已不存在。

File: legged_examples/legged_wl/legged_wl_description/urdf/wl.urdf (robot description, URDF)
Before this commit: robot a1_description, 23 links, 22 joints
Links:
- removed link FL_foot
- removed link FR_foot
- removed link RL_foot
- removed link RR_foot
- added link LF_FOOT, mass 0.037; collision sphere radius=0.025; visual sphere radius=0.01
- added link LH_FOOT, mass 0.037; collision sphere radius=0.025; visual sphere radius=0.01
- added link RF_FOOT, mass 0.037; collision sphere radius=0.025; visual sphere radius=0.01
- added link RH_FOOT, mass 0.037; collision sphere radius=0.025; visual sphere radius=0.01
Joints:
- removed joint FL_foot_fixed
- removed joint FR_foot_fixed
- removed joint RL_foot_fixed
- removed joint RR_foot_fixed
- added joint LF_foot_fixed: type fixed, parent FL_calf, child LF_FOOT, origin xyz=0 0 -0.2 rpy=0 0 0
- added joint LH_foot_fixed: type fixed, parent RL_calf, child LH_FOOT, origin xyz=0 0 -0.2 rpy=0 0 0
- added joint RF_foot_fixed: type fixed, parent FR_calf, child RF_FOOT, origin xyz=0 0 -0.2 rpy=0 0 0
- added joint RH_foot_fixed: type fixed, parent RR_calf, child RH_FOOT, origin xyz=0 0 -0.2 rpy=0 0 0

Commit message: fix(sim): 统一 WL 仿真命名并添加 Docker 启动脚本
原因：WL Gazebo 启动时仍存在 IMU、腿部内部 link 和 self-collision 配置命名未统一的问题，可能导致 LeggedHWSim 找不到 IMU link 并触发 gzserver 段错误。

影响范围：将 WL URDF 的 IMU 统一为 base_imu/base_imu_joint，将腿部内部 link/fixed joint 统一为 LF/RF/LH/RH 前缀，同步 wl/task.info self-collision link pair，给 fixed joint 添加 disableFixedJointLumping，并新增 scripts/docker_launch_ros1.sh 用于启动 Gazebo 或控制器。

验证：精确 rg 检查配置和 URDF 中无 imu_link/imu_joint/unitree_imu 及旧 FL/FR/RL/RR frame 引用；xmllint --noout wl.urdf empty_world.launch；BUILD_TARGETS="legged_wl_description legged_gazebo" scripts/docker_build_ros1.sh；timeout 12s scripts/docker_launch_ros1.sh gazebo -- gui:=false verbose:=true，Gazebo 成功 spawn WL 且无段错误。

File: legged_examples/legged_wl/legged_wl_description/urdf/wl.urdf (robot description, URDF)
Before this commit: robot a1_description, 23 links, 22 joints
Links:
- removed link FL_calf
- removed link FL_hip
- removed link FL_thigh
- removed link FL_thigh_shoulder
- removed link FR_calf
- removed link FR_hip
- removed link FR_thigh
- removed link FR_thigh_shoulder
- removed link RL_calf
- removed link RL_hip
- removed link RL_thigh
- removed link RL_thigh_shoulder
- removed link RR_calf
- removed link RR_hip
- removed link RR_thigh
- removed link RR_thigh_shoulder
- removed link imu_link
- added link LF_calf, mass 0.1394; collision box size=0.02 0.02 0.2; visual mesh filename=../meshes/calf.dae scale=1 1 1
- added link LF_hip, mass 0.6566; visual mesh filename=../meshes/FL_hip.dae scale=1 1 1
- added link LF_thigh, mass 1.1504; collision box size=0.03 0.03 0.2; visual mesh filename=../meshes/thigh_mirror.dae scale=1 1 1
- added link LF_thigh_shoulder
- added link LH_calf, mass 0.1394; collision box size=0.02 0.02 0.2; visual mesh filename=../meshes/calf.dae scale=1 1 1
- added link LH_hip, mass 0.6566; visual mesh filename=../meshes/RL_hip.dae scale=1 1 1
- added link LH_thigh, mass 1.1504; collision box size=0.03 0.03 0.2; visual mesh filename=../meshes/thigh_mirror.dae scale=1 1 1
- added link LH_thigh_shoulder
- added link RF_calf, mass 0.1394; collision box size=0.02 0.02 0.2; visual mesh filename=../meshes/calf.dae scale=1 1 1
- added link RF_hip, mass 0.6566; visual mesh filename=../meshes/FR_hip.dae scale=1 1 1
- added link RF_thigh, mass 1.1504; collision box size=0.03 0.03 0.2; visual mesh filename=../meshes/thigh.dae scale=1 1 1
- added link RF_thigh_shoulder
- added link RH_calf, mass 0.1394; collision box size=0.02 0.02 0.2; visual mesh filename=../meshes/calf.dae scale=1 1 1
- added link RH_hip, mass 0.6566; visual mesh filename=../meshes/RR_hip.dae scale=1 1 1
- added link RH_thigh, mass 1.1504; collision box size=0.03 0.03 0.2; visual mesh filename=../meshes/thigh.dae scale=1 1 1
- added link RH_thigh_shoulder
- added link base_imu, mass 0.001; visual box size=0.001 0.001 0.001
Joints:
- removed joint FL_hip_fixed
- removed joint FR_hip_fixed
- removed joint RL_hip_fixed
- removed joint RR_hip_fixed
- removed joint imu_joint
- added joint LF_hip_fixed: type fixed, parent LF_hip, child LF_thigh_shoulder, origin xyz=0 0.081 0 rpy=0 0 0
- added joint LH_hip_fixed: type fixed, parent LH_hip, child LH_thigh_shoulder, origin xyz=0 0.081 0 rpy=0 0 0
- added joint RF_hip_fixed: type fixed, parent RF_hip, child RF_thigh_shoulder, origin xyz=0 -0.081 0 rpy=0 0 0
- added joint RH_hip_fixed: type fixed, parent RH_hip, child RH_thigh_shoulder, origin xyz=0 -0.081 0 rpy=0 0 0
- added joint base_imu_joint: type fixed, parent trunk, child base_imu, origin xyz=0 0 0 rpy=0 0 0
- joint LF_HAA: child FL_hip -> LF_hip
- joint LF_HFE: child FL_thigh -> LF_thigh; parent FL_hip -> LF_hip
- joint LF_KFE: child FL_calf -> LF_calf; parent FL_thigh -> LF_thigh
- joint LF_foot_fixed: parent FL_calf -> LF_calf
- joint LH_HAA: child RL_hip -> LH_hip
- joint LH_HFE: child RL_thigh -> LH_thigh; parent RL_hip -> LH_hip
- joint LH_KFE: child RL_calf -> LH_calf; parent RL_thigh -> LH_thigh
- joint LH_foot_fixed: parent RL_calf -> LH_calf
- joint RF_HAA: child FR_hip -> RF_hip
- joint RF_HFE: child FR_thigh -> RF_thigh; parent FR_hip -> RF_hip
- joint RF_KFE: child FR_calf -> RF_calf; parent FR_thigh -> RF_thigh
- joint RF_foot_fixed: parent FR_calf -> RF_calf
- joint RH_HAA: child RR_hip -> RH_hip
- joint RH_HFE: child RR_thigh -> RH_thigh; parent RR_hip -> RH_hip
- joint RH_KFE: child RR_calf -> RH_calf; parent RR_thigh -> RH_thigh
- joint RH_foot_fixed: parent RR_calf -> RH_calf

Commit message: fix(rviz): 修复 WL 模型可视化显示
新增基于 OCS2 配置派生的 WL RViz 配置，保留轨迹、GridMap 和目标点工具，同时恢复 RobotModel 不透明显示。

扩展 rviz.launch 的静态模型模式，补充 robot_description、robot_state_publisher、joint_state_publisher 以及 odom 到 base 的静态 TF，便于单独检查 URDF。

补充 grid_map_rviz_plugin 镜像依赖，并调整 WL URDF 的机器人名称、mesh package 路径和材质颜色。

验证：roslaunch --ros-args legged_wl_description rviz.launch publish_static_model:=true。

File: legged_examples/legged_wl/legged_wl_description/urdf/wl.urdf (robot description, URDF)
Before this commit: robot a1_description, 23 links, 22 joints
Links:
- link LF_calf: geometry collision box size=0.02 0.02 0.2; visual mesh filename=package://legged_wl_description/meshes/calf.dae scale=1 1 1
- link LF_hip: geometry visual mesh filename=package://legged_wl_description/meshes/FL_hip.dae scale=1 1 1
- link LF_thigh: geometry collision box size=0.03 0.03 0.2; visual mesh filename=package://legged_wl_description/meshes/thigh_mirror.dae scale=1 1 1
- link LH_calf: geometry collision box size=0.02 0.02 0.2; visual mesh filename=package://legged_wl_description/meshes/calf.dae scale=1 1 1
- link LH_hip: geometry visual mesh filename=package://legged_wl_description/meshes/RL_hip.dae scale=1 1 1
- link LH_thigh: geometry collision box size=0.03 0.03 0.2; visual mesh filename=package://legged_wl_description/meshes/thigh_mirror.dae scale=1 1 1
- link RF_calf: geometry collision box size=0.02 0.02 0.2; visual mesh filename=package://legged_wl_description/meshes/calf.dae scale=1 1 1
- link RF_hip: geometry visual mesh filename=package://legged_wl_description/meshes/FR_hip.dae scale=1 1 1
- link RF_thigh: geometry collision box size=0.03 0.03 0.2; visual mesh filename=package://legged_wl_description/meshes/thigh.dae scale=1 1 1
- link RH_calf: geometry collision box size=0.02 0.02 0.2; visual mesh filename=package://legged_wl_description/meshes/calf.dae scale=1 1 1
- link RH_hip: geometry visual mesh filename=package://legged_wl_description/meshes/RR_hip.dae scale=1 1 1
- link RH_thigh: geometry collision box size=0.03 0.03 0.2; visual mesh filename=package://legged_wl_description/meshes/thigh.dae scale=1 1 1
- link trunk: geometry collision box size=0.286 0.206 0.120; visual mesh filename=package://legged_wl_description/meshes/trunk.dae scale=1 1 1
